File: sch/SX-150 Mk II.brd (EAGLE design)
At the start: 156.2 x 60.6 mm, 189 parts, among them IC1 LM358D, IC2 74HC02D, IC3 LM358D, IC4 LM386M-1, IC5 NJU7096, IC6 REG1117, J1 PJ301M, J2 Line In, Q1 2SC2712, Q10 2SC2712, Q11 2SA1162, Q12 2SC2712, Q13 2SC2712, Q14 2SC2712, Q15 2SC2712, Q16 2SC2712, Q17 2SC2712, Q18 2SC2712, Q19 2SC2712, Q2 2SC2712, Q20 2SC2712, Q21 2SC2712, Q22 2SC2712, Q23 2SC2712, Q24 2SA1162, Q25 2SC2712, Q26 2SC2712, Q27 2SC2712, Q28 2SC2712, Q3 2SC2712, Q4 2SC2712, Q5 2SC2712, Q6 2SC2712, Q7 2SC2712, Q8 2SA1162, Q9 2SC2712, SW1 SP3T, T1 50k, X2 Speaker Out

Commit message: Updating board layout and adding gerbers
Parts:
- FINGERPAD2, PAD1: value FINGERPAD-2A -> GAKKEN-PAD; device dom-key:FINGERPAD-2A -> dom-key:GAKKEN-PAD
- moved TP16 3.42 mm to (140.3, 7.62)
- moved T1 3.24 mm to (121.9, 46.4)
- moved TP7 3.17 mm to (81.9, 48.3)
- moved STRIP- 3.17 mm to (140.3, 3.17)
- moved TP11 2.84 mm to (76.2, 22.9), turned to 0 degrees
- moved C3 2.62 mm to (106.7, 40.0)
- moved R35 2.62 mm to (71.1, 41.3)
- moved C23 2.29 mm to (59.7, 42.5)
- moved R22 2.29 mm to (18.4, 38.1)
- moved R65 2.29 mm to (64.1, 45.7)
- moved TP8 2.29 mm to (66.7, 41.9)
- moved TP10 2.29 mm to (130.2, 10.2)
- moved Q17 2.01 mm to (94.6, 43.8)
- moved Q27 2.01 mm to (107.3, 50.8)
- moved Q28 2.01 mm to (111.1, 50.8)
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Connections:
- net LFO: now also FINGERPAD2.A0, FINGERPAD2.A1; no longer FINGERPAD2.1
- net N$67: now also PAD1.B0, PAD1.B1; no longer PAD1.2
- net N$77: now also PAD1.A0, PAD1.A1; no longer PAD1.1
- net N$82: now also FINGERPAD2.B0, FINGERPAD2.B1; no longer FINGERPAD2.2
Routing:
- net N$67: track 64.6 -> 80.9 mm
- net AGND: track 314.3 -> 300.7 mm, vias 18 -> 19
- net N$77: track 2.54 -> 15.8 mm
- net N$82: track 6.77 -> 19.6 mm
- net LFO: track 114.1 -> 106.0 mm, vias 3 -> 1
- net GND: track 177.7 -> 173.5 mm
- net N$23: track 15.9 -> 12.6 mm
- net N$90: track 6.99 -> 4.22 mm
- net N$35: track 12.6 -> 15.2 mm
- net N$9: track 81.8 -> 79.4 mm
- net +5V: track 378.1 -> 380.2 mm
- net N$18: track 28.6 -> 30.5 mm
- net V+: track 57.4 -> 55.7 mm
- net N$32: track 7.99 -> 6.35 mm
- net N$37: track 11.6 -> 13.2 mm
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Other:
- board size 156.2 x 60.6 mm -> 153.7 x 59.7 mm
- board text added: "+5V"
- board text added: "Atk"
- board text added: "Bat+"
- board text added: "Env"
- board text added: "Gate"
- board text added: "Gnd"
- board text added: "LFO"
- board text added: "Res"
- board text added: "SX-150 Mk II"
- board text added: "Speaker"
- board text added: "Strip"
- board text added: "Tune"
- board text added: "VCF Pad"
- board text added: "VCF-O"
- board text added: "VCF1"
- board text added: "VCF2"
- board text added: "VCO"
- board text added: "VCO Pad"
- board text added: "Vref"
- board text added: "Vref2"

Commit message: Tweaking silkscreen
Parts:
- STRIP+, STRIP-: value TPB1,27 -> TPB2,54; device testpad:B1,27 -> testpad:B2,54
Changed lines of the file:
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@@
 <text x="3.175" y="9.525" size="1.27" layer="25">Strip</text>
 <text x="58.42" y="3.81" size="1.27" layer="25" rot="R180">Speaker</text>
-<text x="59.055" y="17.145" size="1.27" layer="25" rot="R180">Env</text>
+<text x="58.42" y="17.145" size="1.27" layer="25" rot="R180">Env</text>
 <text x="77.47" y="6.35" size="1.27" layer="25">Gate</text>
 <text x="81.28" y="50.8" size="1.27" layer="25">VCO</text>
@@
 <text x="22.86" y="30.48" size="1.27" layer="25">Bat+</text>
 <wire x1="24.765" y1="29.845" x2="26.67" y2="27.305" width="0.254" layer="25"/>
-<text x="26.67" y="21.59" size="1.27" layer="25" rot="R180">Gnd</text>
-<text x="50.8" y="49.53" size="1.27" layer="25">Res</text>
+<text x="26.035" y="20.955" size="1.27" layer="25" rot="R180">Gnd</text>
+<text x="48.895" y="44.45" size="1.27" layer="25">Res</text>
 <text x="43.815" y="42.545" size="1.27" layer="25">VCF1</text>
-<wire x1="46.99" y1="44.45" x2="47.625" y2="46.355" width="0.254" layer="25"/>
+<wire x1="46.99" y1="44.45" x2="48.895" y2="46.355" width="0.254" layer="25"/>
 <text x="52.07" y="40.64" size="1.27" layer="25">VCF2</text>
-<wire x1="53.975" y1="42.545" x2="54.61" y2="43.18" width="0.254" layer="25"/>
+<wire x1="55.245" y1="42.545" x2="55.88" y2="43.18" width="0.254" layer="25"/>
 <text x="67.31" y="39.37" size="1.27" layer="25" rot="R180">Vref2</text>
 <text x="128.27" y="12.7" size="1.27" layer="25">LFO</text>
@@
 <wire x1="133.35" y1="12.7" x2="134.62" y2="12.7" width="0.254" layer="25"/>
 <text x="107.95" y="19.05" size="1.27" layer="25">Strip</text>
-<text x="144.145" y="39.37" size="1.27" layer="25">VCF Pad</text>
-<text x="144.145" y="20.955" size="1.27" layer="25">VCO Pad</text>
+<text x="143.51" y="39.37" size="1.27" layer="25">VCF Pad</text>
+<text x="143.51" y="20.955" size="1.27" layer="25">VCO Pad</text>
 <text x="127.635" y="50.8" size="1.27" layer="25" rot="R270">Tune</text>
 <circle x="40.005" y="30.48" radius="0.898025" width="0.254" layer="25"/>
@@
 <circle x="130.175" y="10.16" radius="0.898025" width="0.254" layer="25"/>
 <circle x="140.335" y="7.62" radius="0.898025" width="0.254" layer="25"/>
-<circle x="140.335" y="3.175" radius="0.898025" width="0.254" layer="25"/>
 <circle x="58.42" y="19.05" radius="0.898025" width="0.254" layer="25"/>
 <circle x="76.2" y="22.86" radius="0.898025" width="0.254" layer="25"/>
 <text x="76.2" y="25.4" size="1.27" layer="25">Atk</text>
+<wire x1="52.07" y1="46.355" x2="51.435" y2="45.72" width="0.254" layer="25"/>
+<wire x1="75.565" y1="23.495" x2="76.2" y2="24.765" width="0.254" layer="25"/>
+<wire x1="109.855" y1="20.955" x2="109.855" y2="20.32" width="0.254" layer="25"/>
+<wire x1="124.46" y1="33.02" x2="123.825" y2="33.655" width="0.254" layer="25"/>
+<wire x1="129.54" y1="10.795" x2="130.175" y2="12.065" width="0.254" layer="25"/>
+<wire x1="67.31" y1="41.275" x2="66.675" y2="40.005" width="0.254" layer="25"/>
+<wire x1="81.28" y1="48.895" x2="81.915" y2="50.165" width="0.254" layer="25"/>
+<wire x1="139.7" y1="8.255" x2="140.335" y2="9.525" width="0.254" layer="25"/>
+<circle x="140.335" y="3.175" radius="1.419903125" width="0.254" layer="25"/>
+<circle x="7.62" y="41.275" radius="1.419903125" width="0.254" layer="25"/>
+<wire x1="59.055" y1="18.415" x2="58.42" y2="17.145" width="0.254" layer="25"/>
+<wire x1="27.305" y1="20.955" x2="26.67" y2="20.32" width="0.254" layer="25"/>
 </plain>
 <attributes>
@@
 <attribute name="POPULARITY" value="73" x="116.84" y="19.05" size="1.778" layer="27" rot="R180" display="off"/>
 <attribute name="SPICEPREFIX" value="C" x="116.84" y="19.05" size="1.778" layer="27" rot="R180" display="off"/>
-<attribute name="NAME" x="114.935" y="19.685" size="0.8128" layer="25" rot="R180"/>
+<attribute name="NAME" x="114.935" y="19.05" size="0.8128" layer="25" rot="R180"/>
 <attribute name="VALUE" x="117.475" y="20.955" size="1.27" layer="27" rot="R180"/>
 </element>
@@
 <attribute name="POPULARITY" value="77" x="88.9" y="52.705" size="1.778" layer="27" rot="R90" display="off"/>
 <attribute name="SPICEPREFIX" value="R" x="88.9" y="52.705" size="1.778" layer="27" rot="R90" display="off"/>
-<attribute name="NAME" x="88.265" y="52.07" size="0.8128" layer="25" rot="R90"/>
+<attribute name="NAME" x="87.63" y="52.07" size="0.8128" layer="25" rot="R90"/>
 <attribute name="VALUE" x="90.805" y="52.07" size="1.27" layer="27" rot="R90"/>
 </element>
@@
 <attribute name="POPULARITY" value="77" x="92.075" y="52.705" size="1.778" layer="27" rot="R90" display="off"/>
 <attribute name="SPICEPREFIX" value="R" x="92.075" y="52.705" size="1.778" layer="27" rot="R90" display="off"/>
-<attribute name="NAME" x="91.44" y="52.07" size="0.8128" layer="25" rot="R90"/>
+<attribute name="NAME" x="93.345" y="53.975" size="0.8128" layer="25" rot="R270"/>
 <attribute name="VALUE" x="93.98" y="52.07" size="1.27" layer="27" rot="R90"/>
 </element>
@@
 </element>
 <element name="D1" library="diode" package="DO41-7.6" value="" x="85.09" y="35.56" smashed="yes" rot="MR90">
-<attribute name="NAME" x="86.741" y="33.528" size="0.8128" layer="26" ratio="10" rot="MR90"/>
+<attribute name="NAME" x="83.82" y="37.465" size="0.8128" layer="26" ratio="10" rot="MR270"/>
 <attribute name="VALUE" x="82.169" y="33.528" size="1.27" layer="28" ratio="10" rot="MR90"/>
 </element>
@@
 <attribute name="POPULARITY" value="14" x="26.035" y="46.99" size="1.778" layer="28" rot="MR0" display="off"/>
 <attribute name="SPICEPREFIX" value="C" x="26.035" y="46.99" size="1.778" layer="28" rot="MR0" display="off"/>
-<attribute name="NAME" x="23.368" y="48.514" size="0.8128" layer="26" ratio="10" rot="MR0"/>
+<attribute name="NAME" x="25.273" y="50.419" size="0.8128" layer="26" ratio="10" rot="MR0"/>
 <attribute name="VALUE" x="23.368" y="44.323" size="1.27" layer="28" ratio="10" rot="MR0"/>
 </element>
@@
 </element>
 <element name="Q21" library="transistor" package="SOT23-BEC" value="2SC2712" x="60.96" y="51.435" smashed="yes" rot="R90">
-<attribute name="NAME" x="61.595" y="49.53" size="0.8128" layer="25" rot="R180"/>
+<attribute name="NAME" x="62.23" y="49.53" size="0.8128" layer="25" rot="R180"/>
 <attribute name="VALUE" x="64.135" y="49.53" size="1.27" layer="27" rot="R90"/>
 </element>
@@
 <attribute name="POPULARITY" value="14" x="26.67" y="38.735" size="1.778" layer="28" rot="MR0" display="off"/>
 <attribute name="SPICEPREFIX" value="C" x="26.67" y="38.735" size="1.778" layer="28" rot="MR0" display="off"/>
-<attribute name="NAME" x="24.003" y="40.259" size="0.8128" layer="26" ratio="10" rot="MR0"/>
+<attribute name="NAME" x="25.908" y="42.164" size="0.8128" layer="26" ratio="10" rot="MR0"/>
 <attribute name="VALUE" x="24.003" y="36.068" size="1.27" layer="28" ratio="10" rot="MR0"/>
 </element>
@@
 </element>
 <element name="LED1" library="led" package="LED3MM" value="" x="17.145" y="23.495" smashed="yes" rot="MR0">
-<attribute name="NAME" x="15.24" y="23.876" size="0.8128" layer="26" ratio="10" rot="MR0"/>
+<attribute name="NAME" x="18.415" y="25.781" size="0.8128" layer="26" ratio="10" rot="MR0"/>
 <attribute name="VALUE" x="15.24" y="21.844" size="1.27" layer="28" ratio="10" rot="MR0"/>
 </element>
@@
 <attribute name="SPICEPREFIX" value="C" x="27.305" y="25.4" size="0.8128" layer="27" rot="R270" display="off"/>
 <attribute name="POPULARITY" value="73" x="27.305" y="25.4" size="0.8128" layer="27" rot="R270" display="off"/>
-<attribute name="NAME" x="27.305" y="23.495" size="0.8128" layer="25" rot="R270"/>
+<attribute name="NAME" x="26.035" y="24.13" size="0.8128" layer="25" rot="R90"/>
 <attribute name="VALUE" x="25.4" y="26.035" size="1.27" layer="27" rot="R270"/>
 </element>
@@
 </element>
 <element name="IC7" library="v-reg" package="TO92-CLP" value="" x="34.29" y="20.32" smashed="yes" rot="MR0">
-<attribute name="NAME" x="32.385" y="20.955" size="0.8128" layer="26" ratio="10" rot="MR0"/>
+<attribute name="NAME" x="31.115" y="20.955" size="0.8128" layer="26" ratio="10" rot="MR0"/>
 <attribute name="VALUE" x="31.115" y="19.05" size="1.27" layer="28" ratio="10" rot="MR0"/>
 </element>
@@
 <attribute name="VALUE" x="65.405" y="3.175" size="1.27" layer="27" rot="R270"/>
 </element>
-<element name="STRIP+" library="testpad" package="B1,27" value="TPB1,27" x="7.62" y="41.275" smashed="yes">
+<element name="STRIP+" library="testpad" package="B2,54" value="TPB2,54" x="7.62" y="41.275" smashed="yes">
 <attribute name="TP_SIGNAL_NAME" value="" x="6.985" y="39.37" size="1" layer="37"/>
-<attribute name="NAME" x="6.985" y="42.291" size="0.8128" layer="25" ratio="10"/>
+<attribute name="NAME" x="6.35" y="42.926" size="0.8128" layer="25" ratio="10"/>
 <attribute name="VALUE" x="6.985" y="40.513" size="0.0254" layer="27"/>
 </element>
-<element name="STRIP-" library="testpad" package="B1,27" value="TPB1,27" x="140.335" y="3.175" smashed="yes">
+<element name="STRIP-" library="testpad" package="B2,54" value="TPB2,54" x="140.335" y="3.175" smashed="yes">
 <attribute name="TP_SIGNAL_NAME" value="" x="139.7" y="1.27" size="1" layer="37"/>
 <attribute name="NAME" x="140.97" y="4.191" size="0.8128" layer="25" ratio="10"/>
@@
 <vertex x="0" y="0"/>
 <vertex x="153.67" y="0"/>
-<vertex x="153.67" y="60.325"/>
-<vertex x="0" y="60.325"/>
+<vertex x="153.67" y="59.69"/>
+<vertex x="0" y="59.69"/>
 </polygon>
 <polygon width="0.4064" layer="16" orphans="yes">
 <vertex x="0" y="0"/>
-<vertex x="154.305" y="0"/>
-<vertex x="154.305" y="60.325"/>
-<vertex x="0" y="60.325"/>
+<vertex x="153.67" y="0"/>
+<vertex x="153.67" y="59.69"/>
+<vertex x="0" y="59.69"/>
 </polygon>
 <contactref element="SW1" pad="4"/>
